Commit message: added lidar urdf

File: src/bullet_envs/turtlebot/urdf/turtlebot.urdf (robot description, URDF)
Before this commit: robot turtlebot, 33 links, 32 joints
Links:
- removed link camera_depth_frame
- removed link camera_depth_optical_frame
- removed link camera_rgb_frame
- removed link camera_rgb_optical_frame
- removed link caster_front_link
- removed link cliff_sensor_front_link
- removed link cliff_sensor_left_link
- removed link cliff_sensor_right_link
- removed link eyes
- removed link gyro_link
- removed link plate_bottom_link
- removed link plate_middle_link
- removed link plate_top_link
- removed link pole_bottom_0_link
- removed link pole_bottom_1_link
- removed link pole_bottom_2_link
- removed link pole_bottom_3_link
- removed link pole_bottom_4_link
- removed link pole_bottom_5_link
- removed link pole_kinect_0_link
- removed link pole_kinect_1_link
- removed link pole_middle_0_link
- removed link pole_middle_1_link
- removed link pole_middle_2_link
- removed link pole_middle_3_link
- removed link pole_top_0_link
- removed link pole_top_1_link
- removed link pole_top_2_link
- removed link pole_top_3_link
- added link base_footprint
- added link base_scan, mass 0.114; collision cylinder length=0.0315 radius=0.055; visual mesh filename=package://turtlebot/meshes/turtlebot3/sensors/lds.stl scale=0.001 0.001 0.001
- added link imu_link
- link base_link: mass 2.4 -> 8.2573504e-01; geometry collision box size=0.140 0.140 0.143; visual mesh filename=package://turtlebot/meshes/turtlebot3/bases/burger_base.stl scale=0.001 0.001 0.001
- link caster_back_link: mass 0.01 -> 0.005; geometry collision box size=0.030 0.009 0.020
- link wheel_left_link: mass 0.1 -> 2.8498940e-02; geometry collision cylinder length=0.018 radius=0.033; visual mesh filename=package://turtlebot/meshes/turtlebot3/wheels/left_tire.stl scale=0.001 0.001 0.001
- link wheel_right_link: mass 0.1 -> 2.8498940e-02; geometry collision cylinder length=0.018 radius=0.033; visual mesh filename=package://turtlebot/meshes/turtlebot3/wheels/right_tire.stl scale=0.001 0.001 0.001
Joints:
- removed joint camera_depth_joint
- removed joint camera_depth_optical_joint
- removed joint camera_joint
- removed joint camera_rgb_joint
- removed joint camera_rgb_optical_joint
- removed joint caster_front_joint
- removed joint cliff_sensor_front_joint
- removed joint cliff_sensor_left_joint
- removed joint cliff_sensor_right_joint
- removed joint gyro_joint
- removed joint plate_bottom_joint
- removed joint plate_middle_joint
- removed joint plate_top_joint
- removed joint pole_bottom_0_joint
- removed joint pole_bottom_1_joint
- removed joint pole_bottom_2_joint
- removed joint pole_bottom_3_joint
- removed joint pole_bottom_4_joint
- removed joint pole_bottom_5_joint
- removed joint pole_kinect_0_joint
- removed joint pole_kinect_1_joint
- removed joint pole_middle_0_joint
- removed joint pole_middle_1_joint
- removed joint pole_middle_2_joint
- removed joint pole_middle_3_joint
- removed joint pole_top_0_joint
- removed joint pole_top_1_joint
- removed joint pole_top_2_joint
- removed joint pole_top_3_joint
- added joint base_joint: type fixed, parent base_footprint, child base_link, origin xyz=0.0 0.0 0.010 rpy=0 0 0
- added joint imu_joint: type fixed, parent base_link, child imu_link, origin xyz=-0.032 0 0.068 rpy=0 0 0
- added joint scan_joint: type fixed, parent base_link, child base_scan, origin xyz=-0.032 0 0.172 rpy=0 0 0
- joint caster_back_joint: origin xyz=-0.135 0.0 0.009 rpy=-1.57079632679 0 0 -> xyz=-0.081 0 -0.004 rpy=-1.57 0 0
- joint wheel_left_joint: origin xyz=0.00 0.115 0.0250 rpy=-1.57079632679 0 0 -> xyz=0.0 0.08 0.023 rpy=-1.57 0 0
- joint wheel_right_joint: origin xyz=0.00 -0.115 0.0250 rpy=-1.57079632679 0 0 -> xyz=0.0 -0.080 0.023 rpy=-1.57 0 0
